File: stepper_driver/m8driver/schematics/m8driver.sch (KiCad schematic (older format))
At the start: 14 parts, among them P1 CHIP2 SOCKET (to LMD), P2 CHIP1 SOCKET (from parport), P3 ISP, Q1 BC547C, X1 16MHz OSC

Commit message: m8driver: Remove reset circuit from schematics
Signed-off-by: Michael Buesch <m@bues.ch>
Parts:
- removed C2: 100u, symbol C
- removed Q1: BC547C, symbol NPN
- removed R1: 4.7k, symbol R
- removed R2: 47k, symbol R
- added C2: 100n, symbol Device:C
- added J1: DEBUG, symbol Connector:Conn_01x01_Female
- C1: symbol C -> Device:CP
- C3: symbol C -> Device:C
- I1: symbol ATMEGA8-16PI -> atmega8x:ATMEGA8-16PI
- P1, P2: symbol DIL24 -> Connector:Conn_01x24_Female
- P3: symbol CONN_3X2 -> Connector:AVR-ISP-6
- R3, R4, R5: symbol R -> Device:R
- X1: symbol CRYSTALOSC -> crystalosc:CRYSTALOSC
Connections:
- wire segments 79 -> 85
Other:
- note removed: "Reset delay"
