File: stepper_driver/estop/schematics/estop.sch (KiCad schematic (older format))
At the start: 21 parts, among them P1 EMC2, P2 ISP, P3 XYZ BRAKE PIN10, P4 SPINDLE, Q1 BC547C, Q2 IRF530, SW1 E-STOP switch

Commit message: estop: Port schematics to new KiCad
Signed-off-by: Michael Buesch <m@bues.ch>
Parts:
- added C4: 100n, symbol Device:C
- C1, C2: symbol C -> Device:CP
- C3: symbol C -> Device:C
- I1: symbol ATMEGA8-16PI -> atmega8x:ATMEGA8-16PI
- P1: symbol CONN_4 -> Connector:Conn_01x04_Female
- P2: symbol CONN_3X2 -> Connector:AVR-ISP-6
- P3: symbol CONN_6 -> Connector:Conn_01x06_Female
- P4: symbol CONN_2 -> Connector:Conn_01x02_Female
- Q1: symbol NPN -> Transistor_BJT:BC547
- Q2: symbol MOS_N -> Transistor_FET:IRF540N
- R1, R10, R2, R3, R4, R5, R6, R7, R8, R9: symbol R -> Device:R
- SW1: symbol SWITCH_INV -> Switch:SW_SPDT
Connections:
- wire segments 70 -> 100
Other:
- note added: "LMD18245\nboard GND"
- note removed: "ODIN board GND"
